Commit message: second commit: lidars, depth camera

File: src/deliverybot_description/urdf/common_properties.xacro (robot description, xacro)
@@ -17,5 +17,17 @@
     <xacro:property name="left_offset_from_steer_y" value="0.03"/>
     <xacro:property name="right_offset_from_steer_y" value="-0.03"/>
-    <xacro:property name="body_wheels_offset_z" value="-0.571468"/>
+    <xacro:property name="body_wheels_offset_z" value="${0.22388 - body_offset_z}"/>
+    <!-- imu-->
+    <xacro:property name="body_imu_offset_z" value="${0.22388 - body_offset_z}"/>
+    <!-- lidar-->
+    <xacro:property name="lidar_offset_x" value="0.72184"/>
+    <xacro:property name="lidar_offset_y" value="0.679109"/>
+    <xacro:property name="lidar_offset_yaw" value="${PI/4}"/>
+    <xacro:property name="body_lidar_offset_z" value="${1.2338 - body_offset_z}"/>
+    <xacro:property name="lidar_sensor_offset_z" value="0.09"/>
+    <!-- depth camera-->
+    <xacro:property name="depth_camera_offset_x" value="0.79739"/>
+    <xacro:property name="depth_camera_offset_y" value="0.0"/>
+    <xacro:property name="body_depth_camera_offset_z" value="${1.3234 - body_offset_z}"/>
     <!-- Ackermann plugin -->
     <xacro:property name="wheelbase_x" value="0.663378"/>

File: src/deliverybot_description/urdf/deliverybot.urdf.xacro (robot description, xacro)
@@ -3,8 +3,13 @@
     <!-- Launch args-->
     <xacro:arg name="use_sensors" default="false"/>
-    <!-- Robot Structure -->
+    <!-- Robot Structure  -->
     <xacro:include filename="$(find deliverybot_description)/urdf/common_properties.xacro" />
     <xacro:include filename="$(find deliverybot_description)/urdf/inertial_properties.xacro" />
     <xacro:include filename="$(find deliverybot_description)/urdf/robot.xacro" />
+    <!-- Sensors-->
+    <xacro:include filename="$(find deliverybot_description)/urdf/imu.xacro" />
+    <xacro:include filename="$(find deliverybot_description)/urdf/lidar.xacro" />
+    <xacro:include filename="$(find deliverybot_description)/urdf/depth_camera.xacro" />
+    <!-- Frictions and Transmissions-->
     <xacro:include filename="$(find deliverybot_description)/urdf/gazebo_properties.xacro" />
     <!-- Ackermann Control -->

File: src/deliverybot_description/urdf/inertial_properties.xacro (robot description, xacro)
@@ -1,4 +1,5 @@
 <?xml version="1.0"?>
 <robot xmlns:xacro="http://www.ros.org/wiki/xacro">
+  <!-- BODY-->
   <xacro:macro name="body_inertial">
       <inertial>
@@ -14,4 +15,5 @@
       </inertial>
   </xacro:macro>
+  <!-- STEERING-->
   <xacro:macro name="steering_inertial">
     <inertial>
@@ -26,4 +28,6 @@
     </inertial>
   </xacro:macro>
+  <!-- WHEELS -->
+  <!-- dummy-->
   <xacro:macro name="cylinder_inertial" params="m r l xyz rpy">
     <inertial>
@@ -35,10 +39,15 @@
     </inertial>
   </xacro:macro>
-  <!-- from cylinder inertial -->
   <xacro:macro name="wheel_right_inertial">
     <inertial>
       <origin rpy="1.57 0 0" xyz="0 0 0"/>
     <mass value="2.26428"/>
-    <inertia ixx="0.142467259859483" ixy="0" ixz="0" iyy="0.142467259859483" iyz="0" izz="0.232177637223095"/>
+    <inertia
+        ixx="0.142467259859483"
+        ixy="0"
+        ixz="0"
+        iyy="0.142467259859483"
+        iyz="0"
+        izz="0.232177637223095"/>
     </inertial>
   </xacro:macro>
@@ -47,6 +56,40 @@
       <origin rpy="1.57 0 0" xyz="0 0 0"/>
       <mass value="2.26428"/>
-      <inertia ixx="0.142467259859483" ixy="0" ixz="0" iyy="0.142467259859483" iyz="0" izz="0.232177637223095"/>
+      <inertia
+        ixx="0.142467259859483"
+        ixy="0"
+        ixz="0"
+        iyy="0.142467259859483"
+        iyz="0"
+        izz="0.232177637223095"/>
     </inertial>
   </xacro:macro>
+  <!-- IMU-->
+  <xacro:macro name="imu_inertial">
+    <inertial>
+      <origin rpy="0.0009 0.0007 0.0003" xyz="0 0 0"/>
+      <mass value="0.011352005096910034"/>
+      <inertia
+        ixx="4.417895181776976e-08"
+        ixy="1.772271240247652e-09"
+        ixz="3.0915776324453116e-10"
+        iyy="2.7136906330486448e-08"
+        iyz="1.9975539330428303e-11"
+        izz="6.995430697342334e-08"/>
+    </inertial>
+  </xacro:macro>
+    <!-- LIDAR -->
+    <xacro:macro name="lidar_inertial">
+      <inertial>
+        <origin rpy="-0.0019 -0.0000 0.0658" xyz="0 0 0"/>
+        <mass value="0.28590020390563653"/>
+        <inertia
+          ixx="0.000762452760169552"
+          ixy="-7.066832712187747e-07"
+          ixz="6.444761162481759e-06"
+          iyy="0.000749768395733118"
+          iyz="6.301900964921601e-07"
+          izz="0.00045580963102950615"/>
+      </inertial>
+    </xacro:macro>
 </robot>

Commit message: third commit: twistmux and safety stop

File: src/deliverybot_description/urdf/common_properties.xacro (robot description, xacro)
@@ -26,4 +26,5 @@
     <xacro:property name="body_lidar_offset_z" value="${1.2338 - body_offset_z}"/>
     <xacro:property name="lidar_sensor_offset_z" value="0.09"/>
+    <xacro:property name="central_lidar_offset_z" value="1.0"/>
     <!-- depth camera-->
     <xacro:property name="depth_camera_offset_x" value="0.79739"/>

File: src/deliverybot_description/urdf/depth_camera.xacro (robot description, xacro)
@@ -20,5 +20,5 @@
         <parent link="depth_camera_link"/>
         <child link="depth_camera_optical_link"/>
-        <origin xyz="0.010 0 0" rpy="${-PI/2} 0 ${-PI/2}"/>
+        <origin xyz="0.011 0 0" rpy="${-PI/2} 0 ${-PI/2}"/>
     </joint>
     <!-- **Higliting differences with normal camera-->

File: src/deliverybot_description/urdf/robot_ros2_control.xacro (robot description, xacro)
@@ -8,5 +8,5 @@
         <parameters>$(find deliverybot_controllers)/config/ackermann_controllers_config.yaml</parameters>
         <ros>
-            <remapping>ackermann_steering_controller/reference:=cmd_vel_stamped</remapping>
+            <remapping>ackermann_steering_controller/reference:=cmd_vel_ack_stamped</remapping>
             <remapping>ackermann_steering_controller/odometry:=odom</remapping>
             <remapping>ackermann_steering_controller/tf_odometry:=tf</remapping>

File: src/deliverybot_description/urdf/velodyne_lidar.xacro (robot description, xacro)
@@ -46,41 +46,41 @@
 <xacro:macro name="lidar_sensor" params="name">
     <gazebo reference="${name}_link">
-        <sensor type="gpu_ray" name="${name}">
+        <sensor name="${name}" type="ray">
+            <always_on>true</always_on>
+            <update_rate>10</update_rate>
+            <visualize>false</visualize>
             <pose>0 0 0 0 0 0</pose>
-            <visualize>false</visualize>
-            <update_rate>5</update_rate>
             <ray>
                 <scan>
-                    <horizontal>
-                        <samples>100</samples>
-                        <resolution>1</resolution>
-                        <min_angle>-1.57</min_angle> <!-- -90 degrees -->
-                        <max_angle>1.57</max_angle>  <!-- 90 degrees -->
-                    </horizontal>
-                    <vertical>
-                        <samples>16</samples>
-                        <resolution>1</resolution>
-                        <min_angle>-0.3044</min_angle> <!-- -17 degrees -->
-                        <max_angle>0.1308</max_angle>  <!-- 7.5 degrees -->
-                    </vertical>
+                <horizontal>
+                    <samples>100</samples>       <!-- The velodyne has 32 beams(samples) -->
+                    <resolution>1</resolution>
+                    <min_angle>-1.5707963</min_angle>
+                    <max_angle>1.5707963</max_angle>
+                </horizontal>
+                <vertical>
+                    <samples>16</samples>       <!-- The velodyne has 32 beams(samples) -->
+                    <resolution>1</resolution>
+                    <min_angle>-0.20</min_angle>
+                    <max_angle>0.06</max_angle>
+                </vertical>
                 </scan>
                 <range>
-                    <min>0.10</min>
-                    <max>20.0</max>
-                    <resolution>0.02</resolution>
+                    <min>0.1</min> <!-- Minimum distance of the beam -->
+                    <max>30.0</max>
+                <resolution>0.01</resolution>
                 </range>
-                <noise>
-                    <type>gaussian</type>
-                    <mean>0.0</mean>
-                    <stddev>0.01</stddev>
-                </noise>
             </ray>
-            <plugin name="gazebo_ros_${name}_controller" filename="libgazebo_ros_ray_sensor.so">
+            <plugin name="gazebo_ros_${name}_velodyne_controller" filename="libgazebo_ros_velodyne_laser.so">
                 <ros>
                     <namespace>/</namespace>
                     <remapping>~/out:=${name}/points</remapping>
                 </ros>
+                <frameName>${name}_link</frameName>
                 <output_type>sensor_msgs/PointCloud2</output_type>
-                <frame_name>${name}_link</frame_name>
+                <min_range>0.1</min_range>
+                <max_range>30</max_range>
+                <min_intensity>0.0</min_intensity>
+                <gaussianNoise>0.0</gaussianNoise>
             </plugin>
         </sensor>

Commit message: fourth commit : laserscan and slam

File: src/deliverybot_description/urdf/common_properties.xacro (robot description, xacro)
@@ -18,4 +18,5 @@
     <xacro:property name="right_offset_from_steer_y" value="-0.03"/>
     <xacro:property name="body_wheels_offset_z" value="${0.22388 - body_offset_z}"/>
+    <!-- scan (2D lidar)-->
     <!-- imu-->
     <xacro:property name="body_imu_offset_z" value="${0.22388 - body_offset_z}"/>
@@ -24,7 +25,7 @@
     <xacro:property name="lidar_offset_y" value="0.679109"/>
     <xacro:property name="lidar_offset_yaw" value="${PI/4}"/>
-    <xacro:property name="body_lidar_offset_z" value="${1.2338 - body_offset_z}"/>
-    <xacro:property name="lidar_sensor_offset_z" value="0.09"/>
-    <xacro:property name="central_lidar_offset_z" value="1.0"/>
+    <xacro:property name="body_lidar_offset_z" value="${1.2194 - body_offset_z}"/>
+    <xacro:property name="lidar_sensor_offset_z" value="${1.3094 - body_offset_z}"/>
+    <xacro:property name="central_lidar_offset_z" value="${1.69712 - body_offset_z}"/>
     <!-- depth camera-->
     <xacro:property name="depth_camera_offset_x" value="0.79739"/>

File: src/deliverybot_description/urdf/depth_camera.xacro (robot description, xacro)
@@ -5,5 +5,5 @@
         <visual>
             <geometry>
-                <box size="0.010 0.03 0.03"/>
+                <box size="0.010 0.3 0.03"/>
             </geometry>
             <material name="white"/>

File: src/deliverybot_description/urdf/inertial_properties.xacro (robot description, xacro)
@@ -93,3 +93,17 @@
       </inertial>
     </xacro:macro>
+    <!-- SCAN (2D LIDAR)-->
+    <xacro:macro name="scan_inertial">
+      <inertial>
+        <origin rpy="0.0330 -0.0053 0.0649" xyz="0 0 0"/>
+        <mass value="0.21203350920404773"/>
+        <inertia
+          ixx="0.011147881277066674"
+          ixy="2.5242109472028173e-05"
+          ixz="-0.0001421632368715965"
+          iyy="0.01111192455712341"
+          iyz="4.152678017456252e-05"
+          izz="0.0006292909214225758"/>
+      </inertial>
+    </xacro:macro>
 </robot>

File: src/deliverybot_description/urdf/lidar.xacro (robot description, xacro)
@@ -3,7 +3,21 @@
     <!-- Links -->
  <!-- Reference link for the fused pointcloud-->
-  <link name="central_lidar_link"/>
+  <link name="central_lidar_link">
+    <xacro:scan_inertial/>
+    <visual>
+        <origin xyz="0 0 0" rpy="0 0 0" />
+        <geometry>
+            <mesh filename="package://deliverybot_description/meshes/scan.obj" />
+        </geometry>
+    </visual>
+    <collision>
+        <origin xyz="0 0 0" rpy="0 0 0" />
+        <geometry>
+            <mesh filename="package://deliverybot_description/meshes/scan.stl" />
+        </geometry>
+    </collision>
+  </link>
   <joint name="body_central_lidar_joint" type="fixed">
-    <origin xyz="0 0 ${body_lidar_offset_z + lidar_sensor_offset_z + central_lidar_offset_z}" rpy="0 0 0" />
+    <origin xyz="0 0 ${central_lidar_offset_z}" rpy="0 0 0" />
         <parent link="body_link" />
         <child link="central_lidar_link" />
@@ -28,11 +42,11 @@
     <link name="${name}_link"/>
     <joint name="${name}_support_joint" type="fixed">
-        <origin xyz="${prefix_x * lidar_offset_x} ${prefix_y * lidar_offset_y} ${-lidar_sensor_offset_z - central_lidar_offset_z}" rpy="0 0 0" />
-        <parent link="central_lidar_link" />
+        <origin xyz="${prefix_x * lidar_offset_x} ${prefix_y * lidar_offset_y} ${body_lidar_offset_z}" rpy="0 0 0" />
+        <parent link="body_link" />
         <child link="${name}_support_link" />
     </joint>
     <joint name="${name}_joint" type="fixed">
-        <origin xyz="${prefix_x * lidar_offset_x} ${prefix_y * lidar_offset_y} ${-central_lidar_offset_z}" rpy="0 0 ${yaw_multiplier * lidar_offset_yaw}" />
-        <parent link="central_lidar_link" />
+        <origin xyz="${prefix_x * lidar_offset_x} ${prefix_y * lidar_offset_y} ${lidar_sensor_offset_z}" rpy="0 0 ${yaw_multiplier * lidar_offset_yaw}" />
+        <parent link="body_link" />
         <child link="${name}_link" />
     </joint>
@@ -55,11 +69,11 @@
                         <samples>100</samples>
                         <resolution>1</resolution>
-                        <min_angle>-1.57</min_angle> <!-- -90 degrees -->
-                        <max_angle>1.57</max_angle>  <!-- 90 degrees -->
+                        <min_angle>-1.04</min_angle> <!-- -60 degrees -->
+                        <max_angle>1.04</max_angle>  <!-- 60 degrees -->
                     </horizontal>
                     <vertical>
-                        <samples>16</samples>
+                        <samples>32</samples>
                         <resolution>1</resolution>
-                        <min_angle>-0.3044</min_angle> <!-- -17 degrees -->
+                        <min_angle>-0.436</min_angle> <!-- -25 degrees -->
                         <max_angle>0.1308</max_angle>  <!-- 7.5 degrees -->
                     </vertical>
@@ -70,9 +84,9 @@
                     <resolution>0.02</resolution>
                 </range>
-                <noise>
+                <!-- <noise>
                     <type>gaussian</type>
                     <mean>0.0</mean>
                     <stddev>0.01</stddev>
-                </noise>
+                </noise> -->
             </ray>
             <plugin name="gazebo_ros_${name}_controller" filename="libgazebo_ros_ray_sensor.so">
