Commit message: gazebo migration

File: src/deliverybot_description/urdf/deliverybot.urdf.xacro (robot description, xacro)
@@ -1,6 +1,23 @@
 <?xml version="1.0"?>
-<robot xmlns:xacro="http://www.ros.org/wiki/xacro" name="deliverybot_robot">
+<robot xmlns:xacro="http://www.ros.org/wiki/xacro" name="deliverybot_sim">
     <!-- Launch args-->
-    <xacro:arg name="use_sensors" default="false"/>
+    <xacro:arg name="gazebo_version" default="ignition"/>
+    <xacro:property name="gazebo_version" value="$(arg gazebo_version)"/>
+    <!-- Gazebo Ignition sensor plugins-->
+    <xacro:if value="${gazebo_version == 'ignition'}">
+      <gazebo>
+        <plugin
+          filename="libignition-gazebo-sensors-system.so" name="ignition::gazebo::systems::Sensors">
+          <render_engine>ogre2</render_engine>
+        </plugin>
+      </gazebo>
+    </xacro:if>
+    <!-- Gazebo gz sensor plugins-->
+    <xacro:if value="${gazebo_version == 'gz'}">
+      <gazebo>
+        <plugin
+          filename="libgazebo_garden_plugin.so" name="gazebo_garden_plugin"/>
+      </gazebo>
+    </xacro:if>
     <!-- Robot Structure  -->
     <xacro:include filename="$(find deliverybot_description)/urdf/common_properties.xacro" />
@@ -14,4 +31,4 @@
     <xacro:include filename="$(find deliverybot_description)/urdf/gazebo_properties.xacro" />
     <!-- Ackermann Control -->
-    <xacro:include filename="$(find deliverybot_description)/urdf/robot_ros2_control.xacro"/>
+    <xacro:include filename="$(find deliverybot_description)/urdf/gazebo_ros2_control.xacro"/>
 </robot>

File: src/deliverybot_description/urdf/depth_camera.xacro (robot description, xacro)
@@ -22,29 +22,98 @@
         <origin xyz="0.011 0 0" rpy="${-PI/2} 0 ${-PI/2}"/>
     </joint>
-    <!-- **Higliting differences with normal camera-->
-    <gazebo reference="depth_camera_link">
-        <material>Gazebo/Red</material>
-        <sensor name="depth_camera" type="depth"> <!-- Depth camera-->
-            <pose> 0 0 0 0 0 0 </pose>
-            <visualize>true</visualize>
-            <update_rate>10</update_rate>
-            <camera>
-                <horizontal_fov>1.089</horizontal_fov>
+    <!-- GAZEBO CLASSIC -->
+    <xacro:if value="${gazebo_version == 'classic'}">
+        <gazebo reference="depth_camera_link">
+            <material>Gazebo/Red</material>
+            <sensor name="depth_camera" type="depth"> <!-- Depth camera-->
+                <pose> 0 0 0 0 0 0 </pose>
+                <visualize>true</visualize>
+                <update_rate>10</update_rate>
+                <camera>
+                    <horizontal_fov>1.089</horizontal_fov>
+                    <image>
+                        <format>B8G8R8</format> <!-- HERE we swap the channels from  RGB to BGR-->
+                        <width>640</width>
+                        <height>480</height>
+                    </image>
+                    <clip>
+                        <near>0.05</near>
+                        <far>8.0</far>
+                    </clip>
+                </camera>
+                <plugin name="camera_controller" filename="libgazebo_ros_camera.so">
+                    <frame_name>depth_camera_optical_link</frame_name>
+                    <min_depth>0.1</min_depth> <!-- Minimum distance from the camera at which objects can be detected - filters out too close objects-->
+                    <max_depth>100.0</max_depth> <!-- Maximum distance from the camera at which objects can be detected - filters out too far objects-->
+                </plugin>
+            </sensor>
+        </gazebo>
+    </xacro:if>
+    <!-- GAZEBO IGNITION AND GZ -->
+    <xacro:if value="${gazebo_version == 'ignition'}">
+        <gazebo reference="depth_camera_link">
+            <sensor type="rgbd_camera" name="depth_camera_sensor">
+            <topic>depth_camera</topic>
+            <frame_id>depth_camera_optical_link</frame_id>
+            <ignition_frame_id>depth_camera_optical_link</ignition_frame_id>
+            <update_rate>20.0</update_rate>
+            <camera name="depth_camera">
+                <horizontal_fov>1.02974</horizontal_fov>
                 <image>
-                    <format>B8G8R8</format> <!-- HERE we swap the channels from  RGB to BGR-->
                     <width>640</width>
                     <height>480</height>
+                    <format>R8G8B8</format>
                 </image>
                 <clip>
-                    <near>0.05</near>
-                    <far>8.0</far>
+                    <near>0.02</near>
+                    <far>20</far>
                 </clip>
             </camera>
-            <plugin name="camera_controller" filename="libgazebo_ros_camera.so">
-                <frame_name>depth_camera_optical_link</frame_name>
-                <min_depth>0.1</min_depth> <!-- Minimum distance from the camera at which objects can be detected - filters out too close objects-->
-                <max_depth>100.0</max_depth> <!-- Maximum distance from the camera at which objects can be detected - filters out too far objects-->
-            </plugin>
-        </sensor>
-    </gazebo>
+            <depth_camera>
+                <clip>
+                    <near>0.02</near>
+                    <far>20</far>
+                </clip>
+            </depth_camera>
+            <point_cloud>
+                <enabled>true</enabled>
+            </point_cloud>
+            <always_on>1</always_on>
+            <visualize>true</visualize>
+            </sensor>
+        </gazebo>
+    </xacro:if>
+    <xacro:if value="${gazebo_version == 'gz'}">
+        <gazebo reference="depth_camera_link">
+            <sensor type="rgbd_camera" name="depth_camera_sensor">
+            <topic>depth_camera</topic>
+            <frame_id>depth_camera_optical_link</frame_id>
+            <gz_frame_id>depth_camera_optical_link</gz_frame_id>
+            <update_rate>20.0</update_rate>
+            <camera name="depth_camera">
+                <horizontal_fov>1.02974</horizontal_fov>
+                <image>
+                    <width>640</width>
+                    <height>480</height>
+                    <format>R8G8B8</format>
+                </image>
+                <clip>
+                <near>0.02</near>
+                <far>20</far>
+                </clip>
+            </camera>
+            <depth_camera>
+                <clip>
+                    <near>0.02</near>
+                    <far>20</far>
+                </clip>
+            </depth_camera>
+            <point_cloud>
+                <enabled>true</enabled>
+            </point_cloud>
+            <always_on>1</always_on>
+            <visualize>true</visualize>
+            </sensor>
+        </gazebo>
+    </xacro:if>
 </robot>

File: src/deliverybot_description/urdf/gazebo_ros2_control.xacro (robot description, xacro)
@@ -1,5 +1,6 @@
 <?xml version="1.0"?>
 <robot xmlns:xacro="http://www.ros.org/wiki/xacro">
-    <!-- Plugin for ROS2 CONTROL -->
+    <!-- GAZEBO CLASSIC -->
+    <xacro:if value="${gazebo_version == 'classic'}">
     <gazebo>
         <plugin filename="libgazebo_ros2_control.so" name="gazebo_ros2_control">
@@ -15,10 +16,59 @@
         </plugin>
     </gazebo>
+    </xacro:if>
+    <!-- GAZEBO IGNITION -->
+    <xacro:if value="${gazebo_version == 'ignition'}">
+    <gazebo>
+        <plugin filename="ign_ros2_control-system" name="ign_ros2_control::IgnitionROS2ControlPlugin">
+        <robot_param>robot_description</robot_param>
+        <robot_param_node>robot_state_publisher</robot_param_node>
+        <parameters>$(find deliverybot_controllers)/config/ackermann_controllers_config.yaml</parameters>
+        <ros>
+            <remapping>ackermann_steering_controller/reference:=cmd_vel_ack_stamped</remapping>
+            <remapping>ackermann_steering_controller/odometry:=odom</remapping>
+            <remapping>ackermann_steering_controller/tf_odometry:=tf</remapping>
+            <robot_base_frame>base_link</robot_base_frame>
+          </ros>
+        </plugin>
+    </gazebo>
+    </xacro:if>
+    <!-- GAZEBO GZ -->
+    <xacro:if value="${gazebo_version == 'gz'}">
+    <gazebo>
+        <plugin filename="gz_ros2_control-system" name="gz_ros2_control::GazeboSimROS2ControlPlugin">
+        <parameters>$(find deliverybot_controllers)/config/ackermann_controllers_config.yaml</parameters>
+         <ros>
+            <remapping>ackermann_steering_controller/reference:=cmd_vel_ack_stamped</remapping>
+            <remapping>ackermann_steering_controller/odometry:=odom</remapping>
+            <remapping>ackermann_steering_controller/tf_odometry:=tf</remapping>
+            <robot_base_frame>base_link</robot_base_frame>
+          </ros>
+        </plugin>
+        <plugin filename="gz-sim-imu-system" name="gz::sim::systems::Imu">
+        </plugin>
+    </gazebo>
+    </xacro:if>
     <!-- Ros2 control -->
-    <ros2_control name="GazeboSystem" type="system">
-        <hardware>
-            <plugin>gazebo_ros2_control/GazeboSystem</plugin>
-        </hardware>
-        <!-- Steering wheels -->
+    <ros2_control name="Gazebo_${gazebo_version}_System" type="system">
+        <!-- GAZEBO CLASSIC-->
+        <xacro:if value="${gazebo_version == 'classic'}">
+            <hardware>
+                <plugin>gazebo_ros2_control/GazeboSystem</plugin>
+            </hardware>
+        </xacro:if>
+         <!-- GAZEBO IGNITION -->
+        <xacro:if value="${gazebo_version == 'ignition'}">
+            <hardware>
+            <plugin>ign_ros2_control/IgnitionSystem</plugin>
+            </hardware>
+        </xacro:if>
+        <!-- GAZEBO GZ-->
+        <xacro:if value="${gazebo_version == 'gz'}">
+            <hardware>
+                <plugin>gz_ros2_control/GazeboSimSystem</plugin>
+            </hardware>
+        </xacro:if>
+        <!-- COMMON INTERFACES  ===================================== -->
+         <!-- Steering wheels -->
         <joint name="steering_left_joint">
             <command_interface name="position">

File: src/deliverybot_description/urdf/imu.xacro (robot description, xacro)
@@ -30,4 +30,8 @@
             <always_on>true</always_on>
             <update_rate>100</update_rate>
+            <!-- GAZEBO IGNITION AND GZ-->
+            <xacro:if value="${gazebo_version == 'gz'}">
+              <gz_frame_id>imu_link</gz_frame_id>
+            </xacro:if>
             <imu>
             <angular_velocity>
@@ -72,5 +76,8 @@
             </linear_acceleration>
             </imu>
-            <plugin name="imu" filename="libgazebo_ros_imu_sensor.so"/> <!-- gazebo plugin-->
+            <!-- GAZEBO CLASSIC PLUGIN -->
+            <xacro:if value="${gazebo_version == 'classic'}">
+              <plugin name="imu" filename="libgazebo_ros_imu_sensor.so"/>
+            </xacro:if>
         </sensor>
     </gazebo>

File: src/deliverybot_description/urdf/lidar.xacro (robot description, xacro)
@@ -58,10 +58,59 @@
 <xacro:lidar_sensor name="lidar_rear_right"  prefix_x="-1" prefix_y="-1" yaw_multiplier="-3"/>
 <!-- Plugins-->
-<xacro:macro name="lidar_sensor" params="name">
-    <gazebo reference="${name}_link">
-        <sensor type="gpu_ray" name="${name}">
-            <pose>0 0 0 0 0 0</pose>
-            <visualize>false</visualize>
-            <update_rate>5</update_rate>
+<xacro:if value="${gazebo_version == 'classic'}">
+    <xacro:macro name="lidar_sensor" params="name">
+        <gazebo reference="${name}_link">
+            <sensor type="gpu_ray" name="${name}">
+                <pose>0 0 0 0 0 0</pose>
+                <visualize>false</visualize>
+                <always_on>true</always_on>
+                <update_rate>5</update_rate>
+                <ray>
+                    <scan>
+                        <horizontal>
+                            <samples>100</samples>
+                            <resolution>1</resolution>
+                            <min_angle>-1.04</min_angle> <!-- -60 degrees -->
+                            <max_angle>1.04</max_angle>  <!-- 60 degrees -->
+                        </horizontal>
+                        <vertical>
+                            <samples>32</samples>
+                            <resolution>1</resolution>
+                            <min_angle>-0.436</min_angle> <!-- -25 degrees -->
+                            <max_angle>0.1308</max_angle>  <!-- 7.5 degrees -->
+                        </vertical>
+                    </scan>
+                    <range>
+                        <min>0.10</min>
+                        <max>20.0</max>
+                        <resolution>0.02</resolution>
+                    </range>
+                    <!-- <noise>
+                        <type>gaussian</type>
+                        <mean>0.0</mean>
+                        <stddev>0.01</stddev>
+                    </noise> -->
+                </ray>
+                <!-- GAZEBO CLASSIC PLUGIN-->
+                <plugin name="gazebo_ros_${name}_controller" filename="libgazebo_ros_ray_sensor.so">
+                    <ros>
+                        <namespace>/</namespace>
+                        <remapping>~/out:=${name}/points</remapping>
+                    </ros>
+                    <output_type>sensor_msgs/PointCloud2</output_type>
+                    <frame_name>${name}_link</frame_name>
+                </plugin>
+            </sensor>
+        </gazebo>
+    </xacro:macro>
+    </xacro:if>
+<xacro:if value="${gazebo_version == 'ignition'}">
+    <xacro:macro name="lidar_sensor" params="name">
+       <gazebo reference="${name}_link">
+        <sensor name="${name}" type="gpu_lidar">
+            <ignition_frame_id>${name}_link</ignition_frame_id>
+            <pose relative_to="${name}_link">0 0 0 0 0 0</pose>
+            <topic>${name}/scan</topic>
+            <update_rate>10</update_rate>
             <ray>
                 <scan>
@@ -84,21 +133,46 @@
                     <resolution>0.02</resolution>
                 </range>
-                <!-- <noise>
-                    <type>gaussian</type>
-                    <mean>0.0</mean>
-                    <stddev>0.01</stddev>
-                </noise> -->
             </ray>
-            <plugin name="gazebo_ros_${name}_controller" filename="libgazebo_ros_ray_sensor.so">
-                <ros>
-                    <namespace>/</namespace>
-                    <remapping>~/out:=${name}/points</remapping>
-                </ros>
-                <output_type>sensor_msgs/PointCloud2</output_type>
-                <frame_name>${name}_link</frame_name>
-            </plugin>
+            <always_on>1</always_on>
+            <visualize>true</visualize>
         </sensor>
     </gazebo>
-</xacro:macro>
+    </xacro:macro>
+    </xacro:if>
+<xacro:if value="${gazebo_version == 'gz'}">
+    <xacro:macro name="lidar_sensor" params="name">
+       <gazebo reference="${name}_link">
+        <sensor name="${name}" type="gpu_lidar">"
+            <ignition_frame_id>"${name}_link</ignition_frame_id>
+            <pose relative_to="${name}_link">0 0 0 0 0 0</pose>
+            <topic>${name}/scan</topic>
+            <update_rate>10</update_rate>
+            <ray>
+                <scan>
+                    <horizontal>
+                        <samples>100</samples>
+                        <resolution>1</resolution>
+                        <min_angle>-1.04</min_angle> <!-- -60 degrees -->
+                        <max_angle>1.04</max_angle>  <!-- 60 degrees -->
+                    </horizontal>
+                    <vertical>
+                        <samples>32</samples>
+                        <resolution>1</resolution>
+                        <min_angle>-0.436</min_angle> <!-- -25 degrees -->
+                        <max_angle>0.1308</max_angle>  <!-- 7.5 degrees -->
+                    </vertical>
+                </scan>
+                <range>
+                    <min>0.10</min>
+                    <max>20.0</max>
+                    <resolution>0.02</resolution>
+                </range>
+            </ray>
+            <always_on>1</always_on>
+            <visualize>true</visualize>
+        </sensor>
+    </gazebo>
+    </xacro:macro>
+    </xacro:if>
 <!-- Use the macro for each LiDAR -->
 <xacro:lidar_sensor name="lidar_front_left"/>
